File: Circuito_impresso.kicad_sch (KiCad schematic)
At the start: 14 parts, among them J1 Extra_inputs, J2 MAX485M/left, J3 MAX485M/right, J4 RPI, Q1 TIP2955, U1 L7805

Commit message: updates to meet requirements; error correction
the width of the tracks is now 0.8 mm (considering the maximum circuit current of 5 amps, with a maximum increase of 40°C; the position of each terminal of the l7805 in the schematic has been corrected; the position of the L7 so that it heatsink does not collide with the TIP

The silkscreen must be done
Parts:
- R1: value 4.7 Ohms -> 3.3 Ohms
Connections:
- net at C1.1, C2.1, J4.2 (Pin_2)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: now also U1.3 (OUT); no longer U1.1 (IN)
- net at C3.1, Q1.1 (B), R1.2: now also U1.1 (IN); no longer U1.3 (OUT)
Changed lines of the file:
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@@
     (in_bom yes) (on_board yes) (fields_autoplaced)
     (property "Reference" "R1" (id 0) (at 225.552 51.054 90))
-    (property "Value" "4.7 Ohms" (id 1) (at 225.552 53.594 90))
+    (property "Value" "3.3 Ohms" (id 1) (at 225.552 53.594 90))
     (property "Footprint" "Resistor_THT:R_Axial_DIN0207_L6.3mm_D2.5mm_P10.16mm_Horizontal" (id 2) (at 225.552 59.182 90)
       (effects (font (size 1.27 1.27)) hide)
@@
     (pin "9")
   )
-  (symbol (lib_id "Regulator_Linear:L7805") (at 200.152 57.404 0) (unit 1)
+  (symbol (lib_id "Regulator_Linear:L7805") (at 200.152 57.404 0) (mirror y) (unit 1)
     (in_bom yes) (on_board yes) (fields_autoplaced)
     (property "Reference" "U1" (id 0) (at 200.152 50.8 0))
     (property "Value" "L7805" (id 1) (at 200.152 53.34 0))
-    (property "Footprint" "AAAA:78XXS" (id 2) (at 200.787 61.214 0)
+    (property "Footprint" "AAAA:78XXS" (id 2) (at 199.517 61.214 0)
       (effects (font (size 1.27 1.27) italic) (justify left) hide)
     )
@@
     )
     (path "/12ada827-2f7e-4eb8-838c-24a7f59b995b"
-      (reference "R1") (unit 1) (value "4.7 Ohms") (footprint "Resistor_THT:R_Axial_DIN0207_L6.3mm_D2.5mm_P10.16mm_Horizontal")
+      (reference "R1") (unit 1) (value "3.3 Ohms") (footprint "Resistor_THT:R_Axial_DIN0207_L6.3mm_D2.5mm_P10.16mm_Horizontal")
     )
     (path "/922bbb59-2217-4cf9-8ac6-d8f99899dc99"

Commit message: Error correction; silkscreen insertion.
The L7805 terminals were inverted on the PCB and have been fixed in this version;

The identification of some of the terminals was made by inserting the serigraphy of the board
Parts:
- renumbered Jn1 to JN4Dba06
Changed lines of the file:
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@@
     (effects (font (size 1.27 1.27)) (justify left bottom))
   )
-  (text "GPIO7" (at 87.376 38.1 90)
+  (text "GPIO8" (at 87.376 38.1 90)
     (effects (font (size 1.27 1.27)) (justify left bottom))
   )
@@
   (symbol (lib_id "Connector_Generic:Conn_01x02") (at 251.206 42.418 0) (mirror y) (unit 1)
     (in_bom yes) (on_board yes)
-    (property "Reference" "Jn1" (id 0) (at 248.158 42.4179 0)
+    (property "Reference" "JN4Dba06" (id 0) (at 248.158 42.4179 0)
       (effects (font (size 1.27 1.27)) (justify left))
     )
@@
       (reference "JIO-1") (unit 1) (value "Conn_01x08") (footprint "Connector_Phoenix_MSTB:PhoenixContact_MSTBA_2,5_8-G_1x08_P5.00mm_Horizontal")
     )
+    (path "/110cbc7e-6a43-407d-889a-e5a40468a9bd"
+      (reference "JN4Dba06") (unit 1) (value "Conn_01x02") (footprint "Connector_Phoenix_MSTB:PhoenixContact_MSTBA_2,5_2-G_1x02_P5.00mm_Horizontal")
+    )
     (path "/c60f47fe-053a-48a8-86e3-26717f4843da"
       (reference "JV1") (unit 1) (value "Conn_01x02") (footprint "Connector_BarrelJack:BarrelJack_Horizontal")
     )
-    (path "/110cbc7e-6a43-407d-889a-e5a40468a9bd"
-      (reference "Jn1") (unit 1) (value "Conn_01x02") (footprint "Connector_Phoenix_MSTB:PhoenixContact_MSTBA_2,5_2-G_1x02_P5.00mm_Horizontal")
-    )
     (path "/ed0c9663-7c30-4dc9-9316-364c94c9c308"
